Commit message: Fixed bugs and added features

File: src/panda_description/urdf/control/panda.ros2_control.xacro (robot description, xacro)
@@ -1,5 +1,5 @@
 <?xml version="1.0"?>
 <robot xmlns:xacro="http://www.ros.org/wiki/xacro">
-    <xacro:macro name="panda_ros2_control" params="name initial_positions_file ros2_control_hardware_type joint_commands_topic_name joint_states_topic_name">
+    <xacro:macro name="panda_ros2_control" params="name prefix initial_positions_file ros2_control_hardware_type">
         <xacro:property name="initial_positions" value="${xacro.load_yaml(initial_positions_file)['initial_positions']}"/>
         <ros2_control name="${name}" type="system">
@@ -10,9 +10,9 @@
                 <xacro:if value="${ros2_control_hardware_type == 'isaac'}">
                     <plugin>topic_based_ros2_control/TopicBasedSystem</plugin>
-                    <param name="joint_commands_topic">${joint_commands_topic_name}</param>
-                    <param name="joint_states_topic">${joint_states_topic_name}</param>
+                    <param name="joint_commands_topic">isaac_joint_commands</param>
+                    <param name="joint_states_topic">isaac_joint_states</param>
                 </xacro:if>
             </hardware>
-            <joint name="panda_joint1">
+            <joint name="${prefix}panda_joint1">
                 <command_interface name="position"/>
                 <state_interface name="position">
@@ -23,5 +23,5 @@
                 </state_interface>
             </joint>
-            <joint name="panda_joint2">
+            <joint name="${prefix}panda_joint2">
                 <command_interface name="position"/>
                 <state_interface name="position">
@@ -32,5 +32,5 @@
                 </state_interface>
             </joint>
-            <joint name="panda_joint3">
+            <joint name="${prefix}panda_joint3">
                 <command_interface name="position"/>
                 <state_interface name="position">
@@ -41,5 +41,5 @@
                 </state_interface>
             </joint>
-            <joint name="panda_joint4">
+            <joint name="${prefix}panda_joint4">
                 <command_interface name="position"/>
                 <state_interface name="position">
@@ -50,5 +50,5 @@
                 </state_interface>
             </joint>
-            <joint name="panda_joint5">
+            <joint name="${prefix}panda_joint5">
                 <command_interface name="position"/>
                 <state_interface name="position">
@@ -59,5 +59,5 @@
                 </state_interface>
             </joint>
-            <joint name="panda_joint6">
+            <joint name="${prefix}panda_joint6">
                 <command_interface name="position"/>
                 <state_interface name="position">
@@ -68,5 +68,5 @@
                 </state_interface>
             </joint>
-            <joint name="panda_joint7">
+            <joint name="${prefix}panda_joint7">
                 <command_interface name="position"/>
                 <state_interface name="position">

File: src/panda_description/urdf/control/panda_hand.ros2_control.xacro (robot description, xacro)
@@ -1,5 +1,5 @@
 <?xml version="1.0"?>
 <robot xmlns:xacro="http://www.ros.org/wiki/xacro">
-    <xacro:macro name="panda_hand_ros2_control" params="name ros2_control_hardware_type joint_commands_topic_name joint_states_topic_name">
+    <xacro:macro name="panda_hand_ros2_control" params="name prefix ros2_control_hardware_type">
         <ros2_control name="${name}" type="system">
             <hardware>
@@ -9,20 +9,10 @@
                 <xacro:if value="${ros2_control_hardware_type == 'isaac'}">
                     <plugin>topic_based_ros2_control/TopicBasedSystem</plugin>
-                    <!-- <param name="joint_commands_topic">/isaac_joint_commands</param>
-                    <param name="joint_states_topic">/isaac_joint_states</param> -->
-                    <param name="joint_commands_topic">${joint_commands_topic_name}</param>
-                    <param name="joint_states_topic">${joint_states_topic_name}</param>
+                    <param name="joint_commands_topic">isaac_joint_commands</param>
+                    <param name="joint_states_topic">isaac_joint_states</param>
                 </xacro:if>
             </hardware>
-            <joint name="panda_finger_joint1">
+            <joint name="${prefix}panda_finger_joint1">
                 <command_interface name="position" />
-                <state_interface name="position">
-                  <param name="initial_value">0.0</param>
-                </state_interface>
-                <state_interface name="velocity">
-                    <param name="initial_value">0.0</param>
-                </state_interface>
-            </joint>
-            <joint name="panda_finger_joint2">
                 <state_interface name="position">
                   <param name="initial_value">0.0</param>

File: src/panda_description/urdf/panda.urdf.xacro (robot description, xacro)
@@ -1,23 +1,21 @@
 <?xml version="1.0"?>
 <robot xmlns:xacro="http://www.ros.org/wiki/xacro" name="panda">
+    <xacro:arg name="prefix" default="" />
     <xacro:arg name="initial_positions_file" default="config/initial_positions.yaml" />
     <xacro:arg name="ros2_control_hardware_type" default="mock_components" />
-    <xacro:arg name="joint_commands_topic_name" default="isaac_joint_commands" />
-    <xacro:arg name="joint_states_topic_name" default="isaac_joint_states" />
-    <!-- Import panda urdf file -->
-    <xacro:include filename="$(find panda_description)/urdf/mech/panda.urdf.xacro" />
-    <!-- Import panda ros2_control description -->
+    <xacro:include filename="$(find panda_description)/urdf/mech/panda_arm.urdf.xacro" />
+    <xacro:include filename="$(find panda_description)/urdf/mech/panda_gripper.urdf.xacro" />
     <xacro:include filename="$(find panda_description)/urdf/control/panda.ros2_control.xacro" />
     <xacro:include filename="$(find panda_description)/urdf/control/panda_hand.ros2_control.xacro" />
+    <xacro:arm prefix="$(arg prefix)" />
+    <xacro:gripper prefix="$(arg prefix)" />
     <xacro:panda_ros2_control name="PandaFakeSystem"
-                                initial_positions_file="$(arg initial_positions_file)"
-                                ros2_control_hardware_type="$(arg ros2_control_hardware_type)"
-                                joint_commands_topic_name="$(arg joint_commands_topic_name)"
-                                joint_states_topic_name="$(arg joint_states_topic_name)"
+                              prefix="$(arg prefix)"
+                              initial_positions_file="$(arg initial_positions_file)"
+                              ros2_control_hardware_type="$(arg ros2_control_hardware_type)"
     />
     <xacro:panda_hand_ros2_control name="PandaHandFakeSystem"
-                                    ros2_control_hardware_type="$(arg ros2_control_hardware_type)"
-                                    joint_commands_topic_name="$(arg joint_commands_topic_name)"
-                                    joint_states_topic_name="$(arg joint_states_topic_name)"
+                                   prefix="$(arg prefix)"
+                                   ros2_control_hardware_type="$(arg ros2_control_hardware_type)"
     />
 </robot>
