Commit message: Restructured project to use a global move_group node

File: src/panda_description/urdf/control/panda_full.ros2_control.xacro (robot description, xacro)
@@ -77,4 +77,13 @@
                 </state_interface>
             </joint>
+            <joint name="${prefix}panda_finger_joint1">
+                <command_interface name="position" />
+                <state_interface name="position">
+                  <param name="initial_value">0.0</param>
+                </state_interface>
+                <state_interface name="velocity">
+                    <param name="initial_value">0.0</param>
+                </state_interface>
+            </joint>
         </ros2_control>
     </xacro:macro>

File: src/panda_description/urdf/control/panda_hand.ros2_control.xacro (robot description, xacro)
@@ -16,5 +16,5 @@
                 <command_interface name="position" />
                 <state_interface name="position">
-                  <param name="initial_value">0.0</param>
+                  <param name="initial_value">0.035</param>
                 </state_interface>
                 <state_interface name="velocity">

File: src/panda_description/urdf/mech/peeler.urdf.xacro (robot description, xacro)
@@ -53,5 +53,5 @@
         </joint>
         <!-- Revolute joint between peeler base and blade -->
-        <joint name="${prefix}blade_joint" type="continuous">
+        <joint name="${prefix}blade_joint" type="fixed">
             <parent link="${prefix}peeler_base"/>
             <child link="${prefix}peeler_blade"/>

File: src/panda_description/urdf/panda.urdf.xacro (robot description, xacro)
@@ -4,18 +4,42 @@
     <xacro:arg name="initial_positions_file" default="config/initial_positions.yaml" />
     <xacro:arg name="ros2_control_hardware_type" default="mock_components" />
+    <xacro:arg name="eef_type" default="gripper" />
     <xacro:include filename="$(find panda_description)/urdf/mech/panda_arm.urdf.xacro" />
-    <xacro:include filename="$(find panda_description)/urdf/mech/panda_gripper.urdf.xacro" />
-    <xacro:include filename="$(find panda_description)/urdf/control/panda.ros2_control.xacro" />
-    <xacro:include filename="$(find panda_description)/urdf/control/panda_hand.ros2_control.xacro" />
+    <xacro:include filename="$(find panda_description)/urdf/control/panda_full.ros2_control.xacro" />
     <xacro:arm prefix="$(arg prefix)" />
-    <xacro:gripper prefix="$(arg prefix)" />
-    <xacro:panda_ros2_control name="PandaFakeSystem"
+    <xacro:property name="eef" value="$(arg eef_type)"/>
+    <xacro:if value="${eef == 'gripper'}">
+        <xacro:include filename="$(find panda_description)/urdf/mech/panda_gripper.urdf.xacro" />
+        <xacro:include filename="$(find panda_description)/urdf/control/panda_full.ros2_control.xacro" />
+        <xacro:gripper prefix="$(arg prefix)" />
+        <xacro:panda_ros2_control_full name="PandaFullFakeSystem"
+                                prefix="$(arg prefix)"
+                                initial_positions_file="$(arg initial_positions_file)"
+                                ros2_control_hardware_type="$(arg ros2_control_hardware_type)" />
+    </xacro:if>
+    <xacro:if value="${eef == 'peeler'}">
+        <xacro:include filename="$(find panda_description)/urdf/mech/peeler.urdf.xacro" />
+        <xacro:include filename="$(find panda_description)/urdf/control/panda.ros2_control.xacro" />
+        <xacro:peeler prefix="$(arg prefix)" parent="panda_link8">
+            <origin xyz="0 0 0" rpy="0 0 0"/>
+        </xacro:peeler>
+        <xacro:panda_ros2_control name="PandaFakeSystem"
+                                    prefix="$(arg prefix)"
+                                    initial_positions_file="$(arg initial_positions_file)"
+                                    ros2_control_hardware_type="$(arg ros2_control_hardware_type)"/>
+    </xacro:if>
+    <xacro:if value="${eef == 'knife'}">
+        <xacro:include filename="$(find panda_description)/urdf/mech/knife.urdf.xacro" />
+        <xacro:include filename="$(find panda_description)/urdf/control/panda.ros2_control.xacro" />
+        <xacro:knife prefix="$(arg prefix)" />
+        <xacro:panda_ros2_control name="PandaFakeSystem"
+                                    prefix="$(arg prefix)"
+                                    initial_positions_file="$(arg initial_positions_file)"
+                                    ros2_control_hardware_type="$(arg ros2_control_hardware_type)"/>
+    </xacro:if>
+    <!-- <xacro:panda_ros2_control name="PandaFakeSystem"
                               prefix="$(arg prefix)"
                               initial_positions_file="$(arg initial_positions_file)"
                               ros2_control_hardware_type="$(arg ros2_control_hardware_type)"
-    />
-    <xacro:panda_hand_ros2_control name="PandaHandFakeSystem"
-                                   prefix="$(arg prefix)"
-                                   ros2_control_hardware_type="$(arg ros2_control_hardware_type)"
-    />
+    /> -->
 </robot>
